File: board/Onboard_Flash.sch (KiCad schematic (older format))
At the start: 10 parts, among them U4 AT25SF641-MHB-T, U5 AT25SF641-MHB-T

Commit message: Fixed the state of the BOM for the PCB being horrid
Parts:
- C19, C20: MFR (none) -> Multicomp; MPN (none) -> MC0603B104J250CT; OC_FARNELL (none) -> 2310559; URL_FARNELL (none) -> https://uk.farnell.com/multicomp/mc0603b104j250ct/cap-0-1-f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
- R4, R5, R6, R7, R8, R9: MFR (none) -> Multicomp; MPN (none) -> MC0063W0603110K; OC_FARNELL (none) -> 2130939; URL_FARNELL (none) -> https://uk.farnell.com/multicomp/mc0063w0603110k/res-10k-1-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
- U4, U5: MFR (none) -> Adesto Technologies; MPN (none) -> AT25SF641-MHB-T; OC_FARNELL (none) -> 2988544; URL_FARNELL (none) -> https://uk.farnell.com/adesto-technologies/at25sf641-mhb-t/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
Changed lines of the file:
@@
 F 1 "AT25SF641-MHB-T" H 3550 3150 50  0000 L CNN
 F 2 "rhais_package-qfn:UDFN-8-1EP_6x5mm_P1.27mm_EP3.4x4mm" H 3500 3200 50  0001 C CNN
-F 3 "" H 3500 3200 50  0001 C CNN
+F 3 "https://www.dialog-semiconductor.com/sites/default/files/at25sf641_111.pdf" H 3500 3200 50  0001 C CNN
+F 4 "Adesto Technologies" H 3500 3500 50  0001 C CNN "MFR"
+F 5 "	AT25SF641-MHB-T" H 3500 3500 50  0001 C CNN "MPN"
+F 6 "2988544" H 3500 3500 50  0001 C CNN "OC_FARNELL"
+F 7 "https://uk.farnell.com/adesto-technologies/at25sf641-mhb-t/flash-memory-64mbit-40-to-85deg/dp/2988544" H 3500 3500 50  0001 C CNN "URL_FARNELL"
 	1    3500 3500
 	1    0    0    -1
@@
 F 1 "AT25SF641-MHB-T" H 7550 3150 50  0000 L CNN
 F 2 "rhais_package-qfn:UDFN-8-1EP_6x5mm_P1.27mm_EP3.4x4mm" H 7500 3200 50  0001 C CNN
-F 3 "" H 7500 3200 50  0001 C CNN
+F 3 "https://www.dialog-semiconductor.com/sites/default/files/at25sf641_111.pdf" H 7500 3200 50  0001 C CNN
+F 4 "Adesto Technologies" H 7500 3500 50  0001 C CNN "MFR"
+F 5 "	AT25SF641-MHB-T" H 7500 3500 50  0001 C CNN "MPN"
+F 6 "2988544" H 7500 3500 50  0001 C CNN "OC_FARNELL"
+F 7 "https://uk.farnell.com/adesto-technologies/at25sf641-mhb-t/flash-memory-64mbit-40-to-85deg/dp/2988544" H 7500 3500 50  0001 C CNN "URL_FARNELL"
 	1    7500 3500
 	1    0    0    -1
@@
 F 1 "0.1uF" H 5092 3455 50  0000 L CNN
 F 2 "rhais_rcl:C0603" H 5000 3500 50  0001 C CNN
-F 3 "~" H 5000 3500 50  0001 C CNN
+F 3 "http://www.farnell.com/datasheets/1870456.pdf" H 5000 3500 50  0001 C CNN
+F 4 "Multicomp" H 5000 3500 50  0001 C CNN "MFR"
+F 5 "MC0603B104J250CT" H 5000 3500 50  0001 C CNN "MPN"
+F 6 "2310559" H 5000 3500 50  0001 C CNN "OC_FARNELL"
+F 7 "https://uk.farnell.com/multicomp/mc0603b104j250ct/cap-0-1-f-25v-5-x7r-0603-reel/dp/2310559" H 5000 3500 50  0001 C CNN "URL_FARNELL"
 	1    5000 3500
 	1    0    0    -1
@@
 F 1 "0.1uF" H 5592 3455 50  0000 L CNN
 F 2 "rhais_rcl:C0603" H 5500 3500 50  0001 C CNN
-F 3 "~" H 5500 3500 50  0001 C CNN
+F 3 "http://www.farnell.com/datasheets/1870456.pdf" H 5500 3500 50  0001 C CNN
+F 4 "Multicomp" H 5500 3500 50  0001 C CNN "MFR"
+F 5 "MC0603B104J250CT" H 5500 3500 50  0001 C CNN "MPN"
+F 6 "2310559" H 5500 3500 50  0001 C CNN "OC_FARNELL"
+F 7 "https://uk.farnell.com/multicomp/mc0603b104j250ct/cap-0-1-f-25v-5-x7r-0603-reel/dp/2310559" H 5500 3500 50  0001 C CNN "URL_FARNELL"
 	1    5500 3500
 	1    0    0    -1
@@
 F 1 "10k" H 6941 3245 50  0000 R CNN
 F 2 "rhais_rcl:R0603" H 7000 3200 50  0001 C CNN
-F 3 "~" H 7000 3200 50  0001 C CNN
+F 3 "http://www.farnell.com/datasheets/1788326.pdf" H 7000 3200 50  0001 C CNN
+F 4 "Multicomp" H 7000 3200 50  0001 C CNN "MFR"
+F 5 "MC0063W0603110K" H 7000 3200 50  0001 C CNN "MPN"
+F 6 "2130939" H 7000 3200 50  0001 C CNN "OC_FARNELL"
+F 7 "https://uk.farnell.com/multicomp/mc0063w0603110k/res-10k-1-0-063w-0603-thick-film/dp/2130939" H 7000 3200 50  0001 C CNN "URL_FARNELL"
 	1    7000 3200
 	1    0    0    1
@@
 F 1 "10k" H 2941 3245 50  0000 R CNN
 F 2 "rhais_rcl:R0603" H 3000 3200 50  0001 C CNN
-F 3 "~" H 3000 3200 50  0001 C CNN
+F 3 "http://www.farnell.com/datasheets/1788326.pdf" H 3000 3200 50  0001 C CNN
+F 4 "Multicomp" H 3000 3200 50  0001 C CNN "MFR"
+F 5 "MC0063W0603110K" H 3000 3200 50  0001 C CNN "MPN"
+F 6 "2130939" H 3000 3200 50  0001 C CNN "OC_FARNELL"
+F 7 "https://uk.farnell.com/multicomp/mc0063w0603110k/res-10k-1-0-063w-0603-thick-film/dp/2130939" H 3000 3200 50  0001 C CNN "URL_FARNELL"
 	1    3000 3200
 	1    0    0    1
@@
 F 1 "10k" V 8025 3400 50  0000 C CNN
 F 2 "rhais_rcl:R0603" H 8100 3400 50  0001 C CNN
-F 3 "~" H 8100 3400 50  0001 C CNN
+F 3 "http://www.farnell.com/datasheets/1788326.pdf" H 8100 3400 50  0001 C CNN
+F 4 "Multicomp" H 8100 3400 50  0001 C CNN "MFR"
+F 5 "MC0063W0603110K" H 8100 3400 50  0001 C CNN "MPN"
+F 6 "2130939" H 8100 3400 50  0001 C CNN "OC_FARNELL"
+F 7 "https://uk.farnell.com/multicomp/mc0063w0603110k/res-10k-1-0-063w-0603-thick-film/dp/2130939" H 8100 3400 50  0001 C CNN "URL_FARNELL"
 	1    8100 3400
 	0    1    1    0
@@
 F 1 "10k" V 8175 3500 50  0000 C CNN
 F 2 "rhais_rcl:R0603" H 8100 3500 50  0001 C CNN
-F 3 "~" H 8100 3500 50  0001 C CNN
+F 3 "http://www.farnell.com/datasheets/1788326.pdf" H 8100 3500 50  0001 C CNN
+F 4 "Multicomp" H 8100 3500 50  0001 C CNN "MFR"
+F 5 "MC0063W0603110K" H 8100 3500 50  0001 C CNN "MPN"
+F 6 "2130939" H 8100 3500 50  0001 C CNN "OC_FARNELL"
+F 7 "https://uk.farnell.com/multicomp/mc0063w0603110k/res-10k-1-0-063w-0603-thick-film/dp/2130939" H 8100 3500 50  0001 C CNN "URL_FARNELL"
 	1    8100 3500
 	0    -1   1    0
@@
 F 1 "10k" V 4025 3400 50  0000 C CNN
 F 2 "rhais_rcl:R0603" H 4100 3400 50  0001 C CNN
-F 3 "~" H 4100 3400 50  0001 C CNN
+F 3 "http://www.farnell.com/datasheets/1788326.pdf" H 4100 3400 50  0001 C CNN
+F 4 "Multicomp" H 4100 3400 50  0001 C CNN "MFR"
+F 5 "MC0063W0603110K" H 4100 3400 50  0001 C CNN "MPN"
+F 6 "2130939" H 4100 3400 50  0001 C CNN "OC_FARNELL"
+F 7 "https://uk.farnell.com/multicomp/mc0063w0603110k/res-10k-1-0-063w-0603-thick-film/dp/2130939" H 4100 3400 50  0001 C CNN "URL_FARNELL"
 	1    4100 3400
 	0    1    1    0
@@
 F 1 "10k" V 4175 3500 50  0000 C CNN
 F 2 "rhais_rcl:R0603" H 4100 3500 50  0001 C CNN
-F 3 "~" H 4100 3500 50  0001 C CNN
+F 3 "http://www.farnell.com/datasheets/1788326.pdf" H 4100 3500 50  0001 C CNN
+F 4 "Multicomp" H 4100 3500 50  0001 C CNN "MFR"
+F 5 "MC0063W0603110K" H 4100 3500 50  0001 C CNN "MPN"
+F 6 "2130939" H 4100 3500 50  0001 C CNN "OC_FARNELL"
+F 7 "https://uk.farnell.com/multicomp/mc0063w0603110k/res-10k-1-0-063w-0603-thick-film/dp/2130939" H 4100 3500 50  0001 C CNN "URL_FARNELL"
 	1    4100 3500
 	0    -1   1    0

Commit message: Cleaned up some loose whitespace in the onboard Flash schematic sheet
Parts:
- U4, U5: MPN AT25SF641-MHB-T -> AT25SF641-MHB-T
Changed lines of the file:
@@
 F 3 "https://www.dialog-semiconductor.com/sites/default/files/at25sf641_111.pdf" H 3500 3200 50  0001 C CNN
 F 4 "Adesto Technologies" H 3500 3500 50  0001 C CNN "MFR"
-F 5 "	AT25SF641-MHB-T" H 3500 3500 50  0001 C CNN "MPN"
+F 5 "AT25SF641-MHB-T" H 3500 3500 50  0001 C CNN "MPN"
 F 6 "2988544" H 3500 3500 50  0001 C CNN "OC_FARNELL"
 F 7 "https://uk.farnell.com/adesto-technologies/at25sf641-mhb-t/flash-memory-64mbit-40-to-85deg/dp/2988544" H 3500 3500 50  0001 C CNN "URL_FARNELL"
@@
 F 3 "https://www.dialog-semiconductor.com/sites/default/files/at25sf641_111.pdf" H 7500 3200 50  0001 C CNN
 F 4 "Adesto Technologies" H 7500 3500 50  0001 C CNN "MFR"
-F 5 "	AT25SF641-MHB-T" H 7500 3500 50  0001 C CNN "MPN"
+F 5 "AT25SF641-MHB-T" H 7500 3500 50  0001 C CNN "MPN"
 F 6 "2988544" H 7500 3500 50  0001 C CNN "OC_FARNELL"
 F 7 "https://uk.farnell.com/adesto-technologies/at25sf641-mhb-t/flash-memory-64mbit-40-to-85deg/dp/2988544" H 7500 3500 50  0001 C CNN "URL_FARNELL"
